Commit message: Update Unity Project to use ROS1 version of UR robot description

File: Assets/urdf/ur10e_rg2.urdf (robot description, URDF)
Before this commit: robot ur10e_rg2, 20 links, 19 joints
Links:
- removed link robot_base
- removed link robot_base_link
- removed link robot_base_link_inertia
- removed link robot_flange
- removed link robot_forearm_link
- removed link robot_ft_frame
- removed link robot_shoulder_link
- removed link robot_tool0
- removed link robot_upper_arm_link
- removed link robot_wrist_1_link
- removed link robot_wrist_2_link
- removed link robot_wrist_3_link
- removed link world
- added link arm_base
- added link arm_base_link
- added link arm_base_link_inertia, mass 4.0; collision mesh filename=package://ur_description/meshes/ur10e/collision/base.stl; visual mesh filename=package://ur_description/meshes/ur10e/visual/base.dae
- added link arm_flange
- added link arm_forearm_link, mass 3.989; collision mesh filename=package://ur_description/meshes/ur10e/collision/forearm.stl; visual mesh filename=package://ur_description/meshes/ur10e/visual/forearm.dae
- added link arm_shoulder_link, mass 7.369; collision mesh filename=package://ur_description/meshes/ur10e/collision/shoulder.stl; visual mesh filename=package://ur_description/meshes/ur10e/visual/shoulder.dae
- added link arm_tcp_link
- added link arm_tool0
- added link arm_upper_arm_link, mass 13.051; collision mesh filename=package://ur_description/meshes/ur10e/collision/upperarm.stl; visual mesh filename=package://ur_description/meshes/ur10e/visual/upperarm.dae
- added link arm_wrist_1_link, mass 2.1; collision mesh filename=package://ur_description/meshes/ur10e/collision/wrist1.stl; visual mesh filename=package://ur_description/meshes/ur10e/visual/wrist1.dae
- added link arm_wrist_2_link, mass 1.98; collision mesh filename=package://ur_description/meshes/ur10e/collision/wrist2.stl; visual mesh filename=package://ur_description/meshes/ur10e/visual/wrist2.dae
- added link arm_wrist_3_link, mass 0.615; collision mesh filename=package://ur_description/meshes/ur10e/collision/wrist3.stl; visual mesh filename=package://ur_description/meshes/ur10e/visual/wrist3.dae
- link gripper_left_inner_finger: geometry collision mesh filename=package://onrobot_rg_description/meshes/rg2/collision/inner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; visual mesh filename=package://onrobot_rg_description/meshes/rg2/visual/inner_fi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
- link gripper_left_inner_knuckle: geometry collision mesh filename=package://onrobot_rg_description/meshes/rg2/collision/inner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; visual mesh filename=package://onrobot_rg_description/meshes/rg2/visual/inner_kn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
- link gripper_left_outer_knuckle: geometry collision mesh filename=package://onrobot_rg_description/meshes/rg2/collision/outer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; visual mesh filename=package://onrobot_rg_description/meshes/rg2/visual/outer_kn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
- link gripper_onrobot_rg2_base_link: geometry collision mesh filename=package://onrobot_rg_description/meshes/rg2/collision/base_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; visual mesh filename=package://onrobot_rg_description/meshes/rg2/visual/base_lin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
- link gripper_right_inner_finger: geometry collision mesh filename=package://onrobot_rg_description/meshes/rg2/collision/inner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; visual mesh filename=package://onrobot_rg_description/meshes/rg2/visual/inner_fi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
- link gripper_right_inner_knuckle: geometry collision mesh filename=package://onrobot_rg_description/meshes/rg2/collision/inner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; visual mesh filename=package://onrobot_rg_description/meshes/rg2/visual/inner_kn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
- link gripper_right_outer_knuckle: geometry collision mesh filename=package://onrobot_rg_description/meshes/rg2/collision/outer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; visual mesh filename=package://onrobot_rg_description/meshes/rg2/visual/outer_kn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
Joints:
- removed joint robot_base_joint
- removed joint robot_base_link-base_fixed_joint
- removed joint robot_base_link-base_link_inertia
- removed joint robot_elbow_joint
- removed joint robot_flange-tool0
- removed joint robot_shoulder_lift_joint
- removed joint robot_shoulder_pan_joint
- removed joint robot_wrist_1_joint
- removed joint robot_wrist_2_joint
- removed joint robot_wrist_3-flange
- removed joint robot_wrist_3_joint
- removed joint robot_wrist_3_link-ft_frame
- added joint arm_base_link-base_fixed_joint: type fixed, parent arm_base_link, child arm_base, origin xyz=0 0 0 rpy=0 0 3.141592653589793
- added joint arm_base_link-base_link_inertia: type fixed, parent arm_base_link, child arm_base_link_inertia, origin xyz=0 0 0 rpy=0 0 3.141592653589793
- added joint arm_elbow_joint: type revolute, parent arm_upper_arm_link, child arm_forearm_link, origin xyz=-0.6127 0 0 rpy=0 0 0, axis 0 0 1, limit lower=-3.141592653589793 upper=3.141592653589793 effort=150.0 velocity=3.141592653589793
- added joint arm_flange-tool0: type fixed, parent arm_flange, child arm_tool0, origin xyz=0 0 0 rpy=1.5707963267948966 0 1.5707963267948966
- added joint arm_shoulder_lift_joint: type revolute, parent arm_shoulder_link, child arm_upper_arm_link, origin xyz=0 0 0 rpy=1.570796327 0 0, axis 0 0 1, limit lower=-6.283185307179586 upper=6.283185307179586 effort=330.0 velocity=2.0943951023931953
- added joint arm_shoulder_pan_joint: type revolute, parent arm_base_link_inertia, child arm_shoulder_link, origin xyz=0 0 0.1807 rpy=0 0 0, axis 0 0 1, limit lower=-6.283185307179586 upper=6.283185307179586 effort=330.0 velocity=2.0943951023931953
- added joint arm_tcp_joint: type fixed, parent arm_tool0, child arm_tcp_link, origin xyz=0 0 0.215 rpy=0 0 0
- added joint arm_wrist_1_joint: type revolute, parent arm_forearm_link, child arm_wrist_1_link, origin xyz=-0.57155 0 0.17415 rpy=0 0 0, axis 0 0 1, limit lower=-6.283185307179586 upper=6.283185307179586 effort=54.0 velocity=3.141592653589793
- added joint arm_wrist_2_joint: type revolute, parent arm_wrist_1_link, child arm_wrist_2_link, origin xyz=0 -0.11985 -2.458164590756244e-11 rpy=1.570796327 0 0, axis 0 0 1, limit lower=-6.283185307179586 upper=6.283185307179586 effort=54.0 velocity=3.141592653589793
- added joint arm_wrist_3-flange: type fixed, parent arm_wrist_3_link, child arm_flange, origin xyz=0 0 0 rpy=0 -1.5707963267948966 -1.5707963267948966
- added joint arm_wrist_3_joint: type revolute, parent arm_wrist_2_link, child arm_wrist_3_link, origin xyz=0 0.11655 -2.390480459346185e-11 rpy=1.570796326589793 3.141592653589793 3.141592653589793, axis 0 0 1, limit lower=-6.283185307179586 upper=6.283185307179586 effort=54.0 velocity=3.141592653589793
- joint ur10e_rg2_connector: origin xyz=0 0 0 rpy=0 1.5707963267948966 0 -> (none); parent robot_flange -> arm_tool0
